File: OptoCounter.kicad_pcb (KiCad board)
At the start: 2 copper layers, 52.4 x 78.4 mm, 50 parts, among them J1 RS-212, J2 PLD-6, J3 USBB-1J, Q1 Q_NPN_BCE, Q2 Q_NPN_BCE, Q3 Q_NPN_BCE, SW1 MSW-11, U1 LM358N, U2 ATMEGA8A-PU, U3 BC56-12SRWA, Y1 8Mhz

Commit message: update
Parts:
- removed R25: 10k, Resistors_THT:R_Axial_DIN0207_L6.3mm_D2.5mm_P10.16mm_Horizontal
- added C8: 330uF, Capacitors_THT:CP_Radial_D6.3mm_P2.50mm, F.Cu at (171.3, 77.0)
- added D4: 1N4734A, MyFootprints:DO-41, F.Cu at (129.3, 83.8)
- C1, C2, C3, C4, C5, C6: footprint Capacitors_THT:C_Disc_D5.0mm_W2.5mm_P5.00mm -> MyFootprints:CAP
- D1, D2: value 1N4007 -> TVS; footprint MyFootprints:1N4007 -> MyFootprints:DO-41
- D3: footprint MyFootprints:1N4007 -> MyFootprints:DO-41
- R1, R10, R11, R12, R13, R14, R15, R16, R17, R18, R19, R2, R20, R21, R22, R23, R24, R26, R27, R28, R3, R4, R5, R6, R7, R8, R9: footprint Resistors_THT:R_Axial_DIN0207_L6.3mm_D2.5mm_P10.16mm_Horizontal -> MyFootprints:RES
- moved R1 5.08 mm to (131.1, 132.8)
- moved R10 5.08 mm to (133.2, 99.4)
- moved R15 5.08 mm to (135.1, 66.6)
- moved R2 5.08 mm to (156.6, 125.1)
- moved R22 5.08 mm to (149.4, 95.4)
- moved R23 5.08 mm to (156.6, 121.7)
- moved R4 5.08 mm to (131.1, 124.1)
- moved R6 5.08 mm to (131.1, 117.3)
- moved R9 5.08 mm to (136.9, 107.4)
- moved R12 5.08 mm to (125.5, 94.9)
- moved R14 5.08 mm to (140.2, 120.1)
- moved R16 5.08 mm to (160.3, 80.0)
- moved R17 5.08 mm to (153.3, 80.0)
- moved R18 5.08 mm to (143.2, 80.0)
- moved R19 5.08 mm to (139.7, 80.0)
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Routing:
- net +5V: track 177.3 -> 184.0 mm
- net Net-(D3-Pad2): track 56.3 -> 54.7 mm
Other:
- net class Default: trace_width 0.25 -> 0.5
- rule pad_to_mask_clearance: 0.1 -> 0.15
- board text added: "AVR ISP"
- board text added: "https://github.com/synthetic65535/OptoCounter"
