File: OptoCounter.sch (KiCad schematic (older format))
At the start: 49 parts, among them J1 RS-212, J2 PLD-6, J3 USBB-1J, Q1 Q_NPN_BCE, Q2 Q_NPN_BCE, Q3 Q_NPN_BCE, SW1 MSW-11, U1 LM358N, U2 ATMEGA8A-PU, U3 BC56-12SRWA, Y1 8Mhz

Commit message: update
Parts:
- removed D1, D2: 1N4007, MyFootprints:1N4007, symbol D_ALT
- added C8: 330uF, Capacitors_THT:CP_Radial_D6.3mm_P2.50mm, symbol CP
- added D1, D2: TVS, MyFootprints:DO-41, symbol D_TVS_ALT
- C1, C2, C3, C4, C5, C6: footprint Capacitors_THT:C_Disc_D5.0mm_W2.5mm_P5.00mm -> MyFootprints:CAP
- D3: footprint MyFootprints:1N4007 -> MyFootprints:DO-41
- D4: footprint (none) -> MyFootprints:DO-41
- R1, R10, R11, R12, R13, R14, R15, R16, R17, R18, R19, R2, R20, R21, R22, R23, R24, R26, R27, R28, R3, R4, R5, R6, R7, R8, R9: footprint Resistors_THT:R_Axial_DIN0207_L6.3mm_D2.5mm_P10.16mm_Horizontal -> MyFootprints:RES
Connections:
- net +5V: now also C8.1, D1.1 (A1)
- net GNDD: now also C8.2, D2.2 (A2)
- net at C1.2, R3.1: now also D1.2 (A2), D2.1 (A1)
Other:
- moved on the sheet: C7, D3, D4, J3, R23, R26
